File: kicad/dm_pcb_batch/dm_pcb_batch.kicad_pcb (KiCad board)
At the start: 2 copper layers, 102.2 x 94.4 mm, 11 parts, among them J1 AVR-ISP-6, Q1 SFH309, SW1 SW_Push, U1 ATtiny85-20P

Commit message: smal fixes ntaa etc
Parts:
- moved C1 92.3 mm to (29.3, 60.7)
- moved D1 92.3 mm to (51.8, 58.3)
- moved Q1 92.3 mm to (51.8, 63.8)
- moved BT1 92.3 mm to (33.7, 47.1)
- moved R1 92.3 mm to (51.7, 33.8)
- moved R2 92.3 mm to (51.7, 37.8)
- moved R3 92.3 mm to (51.7, 41.9)
- moved SW1 92.3 mm to (19.2, 60.7)
- moved U1 92.3 mm to (51.7, 45.9)
- moved J1 92.3 mm to (58.3, 57.9)
- moved LS1 92.3 mm to (53.1, 24.9)
Other:
- board size 102.2 x 94.4 mm -> 136 x 125.3 mm
- board text added: "HELLO"
- board text added: "HIDDEN TEXT"
- board text added: "TEST"

Commit message: smal fixes ntaa etc
Parts:
- added C2: 100n, Capacitor_THT:C_Disc_D3.8mm_W2.6mm_P2.50mm, F.Cu at (184.0, 94.8)
- added D2: LED, LED_THT:LED_D3.0mm, F.Cu at (135.3, 81.4)
- added H1: MountingHole, MountingHole:MountingHole_3.2mm_M3, F.Cu at (174.8, 31.4)
- added H2: MountingHole, MountingHole:MountingHole_3.2mm_M3, F.Cu at (182.2, 139.2)
- added R4: 330, Resistor_THT:R_Axial_DIN0207_L6.3mm_D2.5mm_P10.16mm_Horizontal, F.Cu at (157.3, 81.4)
- R2: value 300 -> 330
- moved D1 177.8 mm to (219.2, 118.2), turned to 130 degrees
- moved C1 173.2 mm to (201.2, 82.8)
- moved R2 167.3 mm to (205.6, 103.4), turned to -50 degrees
- moved LS1 159.7 mm to (185.6, 114.2), turned to 180 degrees
- moved Q1 154.3 mm to (203.7, 36.6)
- moved R3 153.0 mm to (203.8, 58.9), turned to 90 degrees
- moved SW1 144.0 mm to (150.9, 118.9)
- moved J1 143.4 mm to (201.3, 70.0)
- moved BT1 133.7 mm to (167.4, 50.1), turned to 30 degrees
- moved R1 132.0 mm to (177.6, 73.2)
- moved U1 131.8 mm to (179.2, 79.4)
Connections:
- J1 pad 1: BEEP -> MISO
- J1 pad 3: SCK -> BEEP
- U1 pad 6: BEEP -> MISO
- U1 pad 7: SCK -> BEEP
Routing:
- net MISO: track 0.00 -> 62.4 mm
- net PHOTO: track 0.00 -> 58.1 mm
- net BEEP: track 0.00 -> 52.5 mm, vias 0 -> 1
- net Net-(U1-XTAL1/PB3): track 0.00 -> 52.5 mm
- net MOSI: track 0.00 -> 52.3 mm
- net RST: track 0.00 -> 34.2 mm
- net GND: track 0.00 -> 11.2 mm, vias 0 -> 3
- net Net-(D2-A): track 0.00 -> 9.32 mm
- net Net-(D1-A): track 0.00 -> 7.88 mm
- net +3V0: track 0.00 -> 4.05 mm, vias 0 -> 1
- added copper zone on F.Cu, net +3V0
- added copper zone on B.Cu, net GND
Other:
- outline, holes or cut-outs redrawn
- board text added: "algebadge"
- board text added: "hello"
- board text added: "rlfbckr.io"
- board text added: "solder me!"
- board text removed: "HELLO"
- board text removed: "HIDDEN TEXT"
- board text removed: "TEST"
