File: kicad/dm_pcb_batch/dm_pcb_batch.kicad_sch (KiCad schematic)
At the start: 12 parts, among them J1 AVR-ISP-6, J2 Screw_Terminal_01x02, Q1 SFH309, SW1 SW_Push, U1 ATtiny85-20P

Commit message: smal fixes ntaa etc
Parts:
- added C2: 100n, Capacitor_THT:C_Disc_D3.8mm_W2.6mm_P2.50mm, symbol Device:C
- added D2: LED, LED_THT:LED_D3.0mm, symbol Device:LED
- added H1, H2: MountingHole, MountingHole:MountingHole_3.2mm_M3, symbol Mechanical:MountingHole
- added R4: 330, Resistor_THT:R_Axial_DIN0207_L6.3mm_D2.5mm_P10.16mm_Horizontal, symbol Device:R
- R2: value 300 -> 330
Connections:
- net SCK is gone; now on net BEEP: J1.3 (SCK), U1.7 (PB2)
- net +3V0: now also C2.1
- net BEEP: no longer J1.1 (MISO), U1.6 (PB1)
- net GND: now also C2.2, D2.1 (K)
- new net: D2.2 (A), R4.2
- new net MISO: J1.1 (MISO), R4.1, U1.6 (PB1)
